File: v3/scrapyard/active_high_drive/active_high_drive.kicad_pcb (KiCad board)
At the start: 4 copper layers, 11.2 x 26.4 mm, 46 parts, among them J1 Conn_01x10_Pin, Q1 MMDT3904, Q10 MMDT3904, Q11 2N7002DW, Q12 MMDT3904, Q2 2N7002DW, Q3 MMDT3904, Q4 MMDT3904, Q5 2N7002DW, Q6 MMDT3904, Q7 MMDT3904, Q8 2N7002DW, Q9 MMDT3904

Commit message: feat: iterating on v3 design
Parts:
- R1, R10, R11, R12, R13, R14, R15, R16, R17, R18, R19, R2, R20, R21, R22, R23, R24, R3, R4, R5, R6, R7, R8, R9: footprint Resistor_SMD:R_0603_1608Metric -> Resistor_SMD:R_0402_1005Metric
- moved R24 113.3 mm to (0.00, 0.00), turned to 0 degrees
- moved D8 112.5 mm to (0.00, 0.00)
- moved Q12 112.0 mm to (0.00, 0.00), turned to 0 degrees
- moved D7 111.0 mm to (0.00, 0.00)
- moved R23 110.9 mm to (0.00, 0.00)
- moved R22 110.1 mm to (0.00, 0.00)
- moved R21 110.1 mm to (0.00, 0.00)
- moved R15 110.0 mm to (0.00, 0.00), turned to 0 degrees
- moved D6 109.5 mm to (0.00, 0.00)
- moved Q7 108.9 mm to (0.00, 0.00), turned to 0 degrees
- moved Q10 108.9 mm to (0.00, 0.00), turned to 0 degrees
- moved Q11 108.9 mm to (0.00, 0.00)
- moved D5 108.0 mm to (0.00, 0.00)
- moved R14 107.8 mm to (0.00, 0.00)
- moved R19 107.7 mm to (0.00, 0.00)
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Routing:
- net /GND: track 32.8 -> 35.7 mm, vias 13 -> 14
